File: Hardware/ComparatorLogic.kicad_sch (KiCad schematic)
At the start: 20 parts

Commit message: Added 3D models
Parts:
- removed U6: ~, Package_SO:HTSSOP-14-1EP_4.4x5mm_P0.65mm_EP3.4x5mm_Mask3x3.1mm, symbol ComparatorICs:TLV1704AQPWRQ1_
- added R7 (x5): R_Small, symbol Device:R_Small
- added RV7 (x5): R_Potentiometer_Trim, symbol Device:R_Potentiometer_Trim
- added U3: ~, Package_SO:HTSSOP-14-1EP_4.4x5mm_P0.65mm_EP3.4x5mm_Mask3x3.1mm, symbol ComparatorICs:TLV1704AQPWRQ1_
Connections:
- net COMP2A: now also U2.1 (2OUT), U2.13 (4OUT), U2.14 (3OUT), U2.2 (1OUT); no longer U4.1 (2OUT), U4.13 (4OUT), U4.14 (3OUT), U4.2 (1OUT)
- net COMP3A: now also U4.1 (2OUT), U4.13 (4OUT), U4.14 (3OUT), U4.2 (1OUT); no longer U2.1 (2OUT), U2.13 (4OUT), U2.14 (3OUT), U2.2 (1OUT)
- net COMP3_LOGIC: now also U3.3 (VCC); no longer U3.3 (VCC)
- net COMP5A: now also U3.1 (2OUT), U3.13 (4OUT), U3.14 (3OUT), U3.2 (1OUT)
- net COMP5_LOGIC: now also U3.3 (VCC)
- net GND: now also U3.12 (VIN-)
- new net: R7.1, RV7.3 (x5)
Other:
- note added: "Comparator 3"
- note added: "High Treshold"
- note added: "Low Treshold"
- moved on the sheet: R1, R2, R3, R4, R5, R6, R7, RV1, RV2, RV3, RV4, RV5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
