File: Hardware/LogicSelector.kicad_sch (KiCad schematic)
At the start: 6 parts, among them J1 NR01105ANG13-2C

Commit message: Completed Logic Selector page with respec to rotary switches and LED tied to selected voltage levels
Parts:
- added D10, D5, D6, D7, D8, D9: APT1608SEC/J3-AMT, Diode_SMD:D_0603_1608Metric, symbol Device:LED
- added D11, D12, D13, D14, D15, D16: APT1608SECK-AMT, Diode_SMD:D_0603_1608Metric, symbol Device:LED
- added D17, D18, D19, D20, D21, D22: APT1608VRCXF/A-5MAV, Diode_SMD:D_0603_1608Metric, symbol Device:LED
- added D23, D24, D25, D26, D27, D28: SMLEN3WBC8W1, Diode_SMD:D_0603_1608Metric, symbol Device:LED
- added Q1, Q10, Q11, Q12, Q13, Q14, Q15, Q16, Q17, Q18, Q19, Q2, Q20, Q21, Q22, Q23, Q24, Q25, Q26, Q27, Q28, Q29, Q3, Q30, Q31, Q32, Q33, Q34, Q35, Q36, Q37, Q38, Q39, Q4, Q40, Q41, Q42, Q43, Q44, Q45, Q46, Q47, Q48, Q5, Q6, Q7, Q8, Q9: 2SD2653KT146, Package_TO_SOT_SMD:SOT85P240X115-3N, symbol Transistor_BJT:2SD2653KT146
- added R12, R15, R18, R21, R24, R27, R30, R33, R36, R39, R42, R45, R48, R51, R54, R57, R60, R63, R66, R69, R72, R75, R78, R81: 1kΩ, Resistor_SMD:R_0603_1608Metric, symbol Device:R_Small
- added R13, R16, R19, R22, R25, R28, R31, R34, R37, R40, R43, R46, R49, R52, R55, R58, R61, R64, R67, R70, R73, R76, R79, R82: 4.7kΩ, Resistor_SMD:R_0603_1608Metric, symbol Device:R_Small
- added R14, R17, R20, R23, R26, R29, R32, R35, R38, R41, R44, R47, R50, R53, R56, R59, R62, R65, R68, R71, R74, R77, R80, R83: 565 Ω, Resistor_SMD:R_0603_1608Metric, symbol Device:R_Small
- added Z1, Z2, Z3, Z4, Z5, Z6: MM3Z12VT1GX, Diode_SMD:SOD2512X110N, symbol Diode:MM3Z12VT1GX
- added Z10, Z11, Z12, Z7, Z8, Z9: PTZTFTE257.5B, Diode_SMD:PTZTFTE2575B, symbol Diode:PTZTFTE257.5B
- added Z13, Z14, Z15, Z16, Z17, Z18: UDZVTE-174.7B, Diode_SMD:UDZVTE1722B, symbol Diode:UDZVTE-174.7B
- added Z19, Z20, Z21, Z22, Z23, Z24: BZT52H-A3V3-QX, Diode_SMD:SODFL3516X120N, symbol Diode:BZT52H-A3V3-QX
- renumbered J1 to J?
Connections:
- net +12V: now also Q10.1, Q12.1, Q2.1, Q4.1, Q6.1, Q8.1, R13.1, R16.1, R19.1, R22.1, R25.1, R28.1
- net +5V: now also Q26.1, Q28.1, Q30.1, Q32.1, Q34.1, Q36.1, R49.1, R52.1, R55.1, R58.1, R61.1, R64.1
- net +7.5V: now also Q14.1, Q16.1, Q18.1, Q20.1, Q22.1, Q24.1, R31.1, R34.1, R37.1, R40.1, R43.1, R46.1
- net COMP1_LOGIC: now also R12.1, R30.1, R48.1, R66.1
- net COMP2_LOGIC: now also R15.1, R33.1, R51.1, R69.1
- net COMP3_LOGIC: now also R18.1, R36.1, R54.1, R72.1
- net COMP4_LOGIC: now also R21.1, R39.1, R57.1, R75.1
- net COMP5_LOGIC: now also R24.1, R42.1, R60.1, R78.1
- net COMP6_LOGIC: now also R27.1, R45.1, R63.1, R81.1
- new net: Q13.1, Q14.3, R31.2
- new net: Q13.2, Z7.1
- new net: Q13.3, R30.2
- new net: Q16.2, R35.1
- new net: D12.2 (A), R35.2
- new net: Q41.2, Z21.1
- new net: D17.2 (A), R50.2
- new net: Q29.2, Z15.1
- new net: Q3.3, R15.2
- new net: Q3.1, Q4.3, R16.2
- new net: Q31.2, Z16.1
- new net: Q5.2, Z3.1
- new net: Q28.2, R53.1
- new net: D18.2 (A), R53.2
- new net: Q24.2, R47.1
- new net: Q23.1, Q24.3, R46.2
- new net: Q5.3, R18.2
- new net: Q40.2, R71.1
- new net: Q39.1, Q40.3, R70.2
- new net: Q8.2, R23.1
- new net: D8.2 (A), R23.2
- new net: Q25.1, Q26.3, R49.2
- new net: Q27.1, Q28.3, R52.2
- new net: Q27.2, Z14.1
- new net: Q27.3, R51.2
- new net: D19.2 (A), R56.2
- new net: Q1.1, Q2.3, R13.2
- new net: Q19.3, R39.2
- new net: D25.2 (A), R74.2
- new net: Q25.2, Z13.1
- new net: Q25.3, R48.2
- new net: Q18.2, R38.1
- new net: Q17.1, Q18.3, R37.2
- new net: Q31.1, Q32.3, R58.2
- new net: Q48.2, R83.1
- new net: Q47.1, Q48.3, R82.2
- new net: Q47.3, R81.2
- new net: Q37.1, Q38.3, R67.2
- new net: Q37.2, Z19.1
- new net: Q37.3, R66.2
- new net: Q3.2, Z2.1
- new net: Q22.2, R44.1
- new net: Q21.1, Q22.3, R43.2
- new net: D6.2 (A), R17.2
- new net: Q10.2, R26.1
- new net: D9.2 (A), R26.2
- new net: D23.2 (A), R68.2
- new net: Q15.3, R33.2
- new net: Q2.2, R14.1
- new net: Q19.2, Z10.1
- new net: Q15.1, Q16.3, R34.2
- new net: Q34.2, R62.1
- new net: D21.2 (A), R62.2
- new net: Q9.2, Z5.1
- new net: Q36.2, R65.1
- new net: D22.2 (A), R65.2
- new net: Q11.1, Q12.3, R28.2
- new net: D5.2 (A), R14.2
- new net: Q26.2, R50.1
- new net: Q29.1, Q30.3, R55.2
- new net: Q31.3, R57.2
- new net: Q45.2, Z23.1
- new net: Q33.1, Q34.3, R61.2
- new net: D24.2 (A), R71.2
- new net: Q43.1, Q44.3, R76.2
- new net: Q7.1, Q8.3, R22.2
- new net: Q19.1, Q20.3, R40.2
- new net: D16.2 (A), R47.2
- new net: Q14.2, R32.1
- new net: D11.2 (A), R32.2
- new net: Q41.1, Q42.3, R73.2
- new net: Q46.2, R80.1
- new net: D27.2 (A), R80.2
- new net: Q23.2, Z12.1
- new net: Q41.3, R72.2
- new net: Q45.1, Q46.3, R79.2
- new net: Q45.3, R78.2
- new net: Q17.2, Z9.1
- new net: Q9.3, R24.2
- new net: Q29.3, R54.2
- new net: D20.2 (A), R59.2
- new net: Q5.1, Q6.3, R19.2
- new net: Q35.2, Z18.1
- new net: Q1.3, R12.2
- new net: Q32.2, R59.1
- new net: D10.2 (A), R29.2
- new net: Q15.2, Z8.1
- new net: Q11.2, Z6.1
- new net: Q33.2, Z17.1
- new net: Q1.2, Z1.1
- new net: Q21.2, Z11.1
- new net: Q35.1, Q36.3, R64.2
- new net: Q35.3, R63.2
- new net: Q11.3, R27.2
- new net: Q39.2, Z20.1
- new net: D26.2 (A), R77.2
- new net: Q20.2, R41.1
- new net: Q12.2, R29.1
- new net: Q44.2, R77.1
- new net: Q47.2, Z24.1
- new net: Q4.2, R17.1
- new net: Q42.2, R74.1
- new net: D14.2 (A), R41.2
- new net: Q17.3, R36.2
- new net: Q39.3, R69.2
- new net: Q30.2, R56.1
- new net: Q10.3, Q9.1, R25.2
- new net: Q23.3, R45.2
- new net: Q6.2, R20.1
- new net: D7.2 (A), R20.2
- new net: D28.2 (A), R83.2
- new net: Q43.3, R75.2
- new net: Q7.2, Z4.1
- new net: Q33.3, R60.2
- new net: Q21.3, R42.2
- new net: Q43.2, Z22.1
- new net: D13.2 (A), R38.2
- new net: D15.2 (A), R44.2
- new net: Q38.2, R68.1
- new net: Q7.3, R21.2
- new net +3V3: Q38.1, Q40.1, Q42.1, Q44.1, Q46.1, Q48.1, R67.1, R70.1, R73.1, R76.1, R79.1, R82.1
- new net GND: D10.1 (K), D11.1 (K), D12.1 (K), D13.1 (K), D14.1 (K), D15.1 (K), D16.1 (K), D17.1 (K), D18.1 (K), D19.1 (K), D20.1 (K), D21.1 (K), D22.1 (K), D23.1 (K), D24.1 (K), D25.1 (K), D26.1 (K), D27.1 (K), D28.1 (K), D5.1 (K), D6.1 (K), D7.1 (K), D8.1 (K), D9.1 (K), Z1.2, Z10.2, Z11.2, Z12.2, Z13.2, Z14.2, Z15.2, Z16.2, Z17.2, Z18.2, Z19.2, Z2.2, Z20.2, Z21.2, Z22.2, Z23.2, Z24.2, Z3.2, Z4.2, Z5.2, Z6.2, Z7.2, Z8.2, Z9.2
Other:
- note added: "11.8v Bias Set"
- note added: "12v Turn-On"
- note added: "3.3v Turn-On"
- note added: "5v Turn-On"
- note added: "7.5v Bias Set"
- note added: "7.5v Turn-On"
- note added: "Blue LED"
- note added: "Orange LED"
- note added: "Red LED"
- note added: "Violet LED"
- note added: "White LED"
- moved on the sheet: J?

Commit message: Added changes to logic side for comparator inputs
Parts:
- added TP6: Comp1_Logic, TestPoint:TestPoint_Keystone_5015_Micro-Minature, symbol Connector:TestPoint_Flag
- added TP6: Comp4_Logic, TestPoint:TestPoint_Keystone_5015_Micro-Minature, symbol Connector:TestPoint_Flag
- added TP6: Comp3_Logic, TestPoint:TestPoint_Keystone_5015_Micro-Minature, symbol Connector:TestPoint_Flag
- added TP6: Comp2_Logic, TestPoint:TestPoint_Keystone_5015_Micro-Minature, symbol Connector:TestPoint_Flag
- added TP6: Comp5_Logic, TestPoint:TestPoint_Keystone_5015_Micro-Minature, symbol Connector:TestPoint_Flag
- added TP6: Comp6_Logic, TestPoint:TestPoint_Keystone_5015_Micro-Minature, symbol Connector:TestPoint_Flag
Connections:
- net COMP1_LOGIC: now also TP6.1
- net COMP2_LOGIC: now also TP6.1
- net COMP3_LOGIC: now also TP6.1
- net COMP4_LOGIC: now also TP6.1
- net COMP5_LOGIC: now also TP6.1
- net COMP6_LOGIC: now also TP6.1
