File: Hardware/UTCB.kicad_pcb (KiCad board)
At the start: 4 copper layers, 101.6 x 135.4 mm, 89 parts, among them IC1 TR05S3V3, J1 Conn_01x02, J10 Conn_01x06, SW1 SW_DIP_x06

Commit message: Completed rev1.0 traces
Finished traces
Parts:
- moved TP2 4.28 mm to (127.8, 105.2)
- moved TP3 2.33 mm to (130.9, 140.7)
- moved R9 0.25 mm to (190.7, 34.0), turned to 0 degrees
Routing:
- net COMP6A: track 13.0 -> 149.2 mm, vias 0 -> 1
- net COMP3A: track 14.8 -> 140.6 mm, vias 0 -> 1
- net COMP2A: track 8.07 -> 108.7 mm, vias 0 -> 1
- net COMP5A: track 13.2 -> 110.9 mm, vias 0 -> 1
- net COMP1A: track 10.1 -> 76.6 mm
- net Signal6: track 182.4 -> 234.1 mm, vias 0 -> 2
- net COMP4A: track 13.5 -> 63.6 mm, vias 0 -> 1
- net /ComparatorLogic/COMP6_LOW: track 0.00 -> 45.8 mm, vias 0 -> 1
- net /ComparatorLogic/COMP3_HIGH: track 0.00 -> 39.1 mm, vias 0 -> 1
- net /ComparatorLogic/Timing6Check: track 0.00 -> 36.8 mm
- net /ComparatorLogic/COMP5_LOW: track 7.39 -> 42.5 mm, vias 0 -> 1
- net /ComparatorLogic/COMP2_HIGH: track 21.3 -> 55.6 mm
- net /ComparatorLogic/COMP2_LOW: track 0.00 -> 32.8 mm
- net /ComparatorLogic/COMP3_LOW: track 0.00 -> 31.7 mm
- net /ComparatorLogic/Failure_Output: track 0.00 -> 28.4 mm
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- added copper zone on In2.Cu, net +12V
- added copper zone on F.Cu, net +3.3V

Commit message: Minor modifications
Added 3D model for the regulator, updated to socket for signal inputs, and updated to power pours for certain PWR pins.
Parts:
- J10: footprint Connector_PinHeader_1.27mm:PinHeader_1x06_P1.27mm_Vertical -> Connector_PinSocket_1.27mm:PinSocket_1x06_P1.27mm_Vertical
- moved TP33 4.51 mm to (190.4, 33.5)
- moved TP26 4.15 mm to (184.7, 69.8)
- moved R9 4.10 mm to (192.2, 37.8)
- moved TP7 3.42 mm to (105.9, 69.6)
- moved TP4 3.37 mm to (166.1, 74.4)
- moved TP24 3.04 mm to (157.7, 68.6)
- moved TP25 2.92 mm to (170.4, 68.6)
- moved TP2 2.33 mm to (127.0, 107.4)
- moved TP14 2.03 mm to (107.2, 137.9)
- moved TP23 1.98 mm to (136.7, 137.2)
- moved TP15 1.82 mm to (121.4, 137.7)
- moved TP8 1.80 mm to (121.2, 67.8)
- moved TP9 1.52 mm to (135.4, 67.3)
Routing:
- net /ComparatorLogic/COMP2_HIGH: track 55.6 -> 42.0 mm, vias 0 -> 1
- net /ComparatorLogic/Failure_Output: track 28.4 -> 33.2 mm
- net /ComparatorLogic/COMP1_HIGH: track 42.2 -> 46.8 mm
- net /ComparatorLogic/COMP4_HIGH: track 30.0 -> 34.4 mm
- net COMP4A: track 63.6 -> 67.6 mm
- net /ComparatorLogic/COMP3_HIGH: track 39.1 -> 43.0 mm
- net /ComparatorLogic/COMP1_LOW: track 31.6 -> 35.4 mm
- net /ComparatorLogic/COMP4_LOW: track 45.9 -> 49.5 mm
- net /ComparatorLogic/Timing1Check: track 28.9 -> 31.5 mm
- net /ComparatorLogic/Timing4Check: track 41.0 -> 42.8 mm
- net /ComparatorLogic/COMP2_LOW: track 32.8 -> 34.0 mm
- net /ComparatorLogic/COMP3_LOW: track 31.7 -> 32.6 mm
- net Signal2: track 139.0 -> 138.3 mm
Other:
- board text added: "Comparator 1"
- board text added: "Comparator 2"
- board text added: "Comparator 3"
- board text added: "Comparator 4"
- board text added: "Comparator 5"
- board text added: "Comparator 6"
- board text removed: "Comparator 1 Logic"
- board text removed: "Comparator 2 Logic"
- board text removed: "Comparator 3 Logic"
- board text removed: "Comparator 4 Logic"
- board text removed: "Comparator 5 Logic"
- board text removed: "Comparator 6 Logic"
